Commit message: working out pybullet stuff

File: simulation_env/assets/biped2d_pybullet.urdf (robot description, URDF)
Before this commit: robot balance, 11 links, 10 joints
Links:
- removed link x_prismatic
- link y_prismatic: mass 70 -> 0.01
- link z_prismatic: mass 70 -> 0.01
Joints:
- removed joint torso_to_x
- removed joint x_to_z
- added joint torso_to_z: type continuous, parent z_prismatic, child torso, origin xyz=0 0 1.4 rpy=0 0 0, axis 1 0 0
