Commit message: biped working

File: simulation_env/assets/biped_custum2.urdf (robot description, URDF)
Before this commit: robot balance, 10 links, 9 joints
Links:
- removed link world
- added link x_prismatic, mass 10
- link y_prismatic: mass 0 -> 10
- link z_prismatic: mass 0 -> 10
Joints:
- removed joint torso_to_z
- removed joint y_to_world
- removed joint z_to_y
- added joint Torso_to_x: type prismatic, parent torso, child x_prismatic, origin xyz=0 0 0 rpy=0 0 0, axis 1 0 0, limit lower=1 upper=-1 effort=0.0 velocity=1000.0
- added joint Torso_to_y: type prismatic, parent torso, child y_prismatic, origin xyz=0 0 0 rpy=0 0 0, axis 0 1 0, limit lower=1 upper=-1 effort=0.0 velocity=1000.0
- added joint Torso_to_z: type prismatic, parent torso, child z_prismatic, origin xyz=0 0 0 rpy=0 0 0, axis 0 0 1, limit lower=1 upper=-1 effort=0.0 velocity=1000.0
