Commit message: model finished

File: simulation_env/assets/biped_norotation_zfixed.urdf (robot description, URDF)
Before this commit: robot balance, 10 links, 9 joints
Links:
- added link head, mass 70; collision cylinder length=0.05 radius=0.07; visual cylinder length=0.05 radius=0.07
- added link origin, mass 0; visual box size=0.1 0.1 0.1
- link x_prismatic: mass 10 -> 0
- link y_prismatic: mass 10 -> 0
- link z_prismatic: mass 10 -> 0
Joints:
- removed joint Torso_to_x
- removed joint Torso_to_y
- removed joint Torso_to_z
- added joint neck_joint: type fixed, parent head, child torso, origin xyz=0 0 0 rpy=0 0 0, axis 0 0 0, limit lower=1 upper=-1 effort=0.0 velocity=1000.0
- added joint origin_to_z: type fixed, parent origin, child z_prismatic, origin xyz=0 0 0 rpy=0 0 0, axis 0 0 1, limit lower=1 upper=-1 effort=0.0 velocity=1000.0
- added joint x_to_y: type prismatic, parent x_prismatic, child y_prismatic, origin xyz=0 0 0 rpy=0 0 0, axis 0 1 0, limit lower=1 upper=-1 effort=0.0 velocity=1000.0
- added joint y_to_head: type fixed, parent y_prismatic, child head, origin xyz=0 0 0 rpy=0 0 0, axis 0 0 0, limit lower=1 upper=-1 effort=0.0 velocity=1000.0
- added joint z_to_x: type prismatic, parent z_prismatic, child x_prismatic, origin xyz=0 0 0 rpy=0 0 0, axis 1 0 0, limit lower=1 upper=-1 effort=0.0 velocity=1000.0
