Commit message: training program started, WIP

File: simulation_env/assets/biped_norotation_2d.urdf (robot description, URDF)
Before this commit: robot balance, 12 links, 11 joints
Links:
- added link l_legrot, mass 5
- added link r_legrot, mass 5
- link head: mass 70 -> 10
Joints:
- removed joint torso_to_leftleg
- removed joint torso_to_rightleg
- added joint rot_to_leftleg: type revolute, parent l_legrot, child l_upperleg, origin xyz=-0.05 0 -0.17 rpy=0 0 0, axis 1 0 0, limit lower=-1.57. upper=1.57 effort=10.0 velocity=1000.0
- added joint rot_to_rightleg: type revolute, parent r_legrot, child r_upperleg, origin xyz=0.05 0 -0.17 rpy=0 0 0, axis 1 0 0, limit lower=-1.57. upper=1.57 effort=0.0 velocity=1000.0
- added joint torso_to_l_legrot: type revolute, parent torso, child l_legrot, origin xyz=-0.03 0 0 rpy=0 0 0, axis 0 1 0, limit lower=-0.125 upper=0.125 effort=0.0 velocity=1000.0
- added joint torso_to_r_legrot: type revolute, parent torso, child r_legrot, origin xyz=0.03 0 0 rpy=0 0 0, axis 0 1 0, limit lower=-0.125 upper=0.125 effort=0.0 velocity=1000.0
- joint l_ankle: origin xyz=-0.05 -0.03 -.459 rpy=0 0 0 -> xyz=-0.05 -0.03 -.43 rpy=0 0 0
- joint r_ankle: origin xyz=0.05 -0.03 -.459 rpy=0 0 0 -> xyz=0.05 -0.03 -.43 rpy=0 0 0
