Commit message: all models made and fixed

File: simulation_env/assets/biped_freeman.urdf (robot description, URDF)
Before this commit: robot balance, 12 links, 11 joints
Links:
- added link l_legrot, mass 5
- added link r_legrot, mass 5
- link head: mass 70 -> 10
Joints:
- removed joint torso_to_leftleg
- removed joint torso_to_rightleg
- added joint rot_to_leftleg: type revolute, parent l_legrot, child l_upperleg, origin xyz=-0.05 0 -0.17 rpy=0 0 0, axis 1 0 0, limit lower=-1.57. upper=1.57 effort=10.0 velocity=1000.0
- added joint rot_to_rightleg: type revolute, parent r_legrot, child r_upperleg, origin xyz=0.05 0 -0.17 rpy=0 0 0, axis 1 0 0, limit lower=-1.57. upper=1.57 effort=0.0 velocity=1000.0
- added joint torso_to_l_legrot: type revolute, parent torso, child l_legrot, origin xyz=-0.03 0 0 rpy=0 0 0, axis 0 1 0, limit lower=-0.125 upper=0.125 effort=0.0 velocity=1000.0
- added joint torso_to_r_legrot: type revolute, parent torso, child r_legrot, origin xyz=0.03 0 0 rpy=0 0 0, axis 0 1 0, limit lower=-0.125 upper=0.125 effort=0.0 velocity=1000.0
- joint l_ankle: origin xyz=-0.05 -0.03 -.459 rpy=0 0 0 -> xyz=-0.05 -0.03 -.43 rpy=0 0 0
- joint origin_to_z: type fixed -> prismatic
- joint r_ankle: origin xyz=0.05 -0.03 -.459 rpy=0 0 0 -> xyz=0.05 -0.03 -.43 rpy=0 0 0

File: simulation_env/assets/biped_norotation_2d.urdf (robot description, URDF)
Before this commit: robot balance, 10 links, 9 joints
Links:
- removed link world
- added link head, mass 70; collision cylinder length=0.05 radius=0.07; visual cylinder length=0.05 radius=0.07
- added link origin, mass 0; visual box size=0.1 0.1 0.1
- added link x_prismatic, mass 0
- link y_prismatic: mass 0.01 -> 0
- link z_prismatic: mass 0.01 -> 0
Joints:
- removed joint torso_to_z
- removed joint y_to_world
- removed joint z_to_y
- added joint neck_joint: type fixed, parent head, child torso, origin xyz=0 0 0 rpy=0 0 0, axis 0 0 0, limit lower=1 upper=-1 effort=0.0 velocity=1000.0
- added joint origin_to_z: type prismatic, parent origin, child z_prismatic, origin xyz=0 0 0 rpy=0 0 0, axis 0 0 1, limit lower=1 upper=-1 effort=0.0 velocity=1000.0
- added joint x_to_y: type prismatic, parent x_prismatic, child y_prismatic, origin xyz=0 0 0 rpy=0 0 0, axis 0 1 0, limit lower=1 upper=-1 effort=0.0 velocity=1000.0
- added joint y_to_head: type fixed, parent y_prismatic, child head, origin xyz=0 0 0 rpy=0 0 0, axis 0 0 0, limit lower=1 upper=-1 effort=0.0 velocity=1000.0
- added joint z_to_x: type prismatic, parent z_prismatic, child x_prismatic, origin xyz=0 0 0 rpy=0 0 0, axis 1 0 0, limit lower=1 upper=-1 effort=0.0 velocity=1000.0

Commit message: minor corrections

File: simulation_env/assets/biped_freeman.urdf (robot description, URDF)
Before this commit: robot balance, 14 links, 13 joints
Joints:
- joint y_to_head: type fixed -> prismatic
