Commit message: fixed a bunch of training errors, including the starting position, activation functions, control mode and intial pop weights

File: simulation_env/assets/biped_freeman_simple.urdf (robot description, URDF)
Before this commit: robot balance, 12 links, 11 joints
Joints:
- joint l_knee: limit lower=-1.57. upper=1.57 effort=10.0 velocity=1000.0 -> lower=-1.57. upper=0.2 effort=10.0 velocity=1000.0
- joint r_knee: limit lower=-1.57. upper=1.57 effort=10.0 velocity=1000.0 -> lower=-1.57. upper=0.2 effort=10.0 velocity=1000.0

File: simulation_env/assets/plane.urdf (robot description, URDF)
Before this commit: robot plane, 1 links, 0 joints
Links:
- added link origin, mass 0; visual box size=0.1 0.1 0.1
Joints:
- added joint plane_to_origin: type fixed, parent origin, child planeLink, origin xyz=0 0 0 rpy=0 0 0
