Commit message: error correction + attempt at 3d training

File: simulation_env/assets/biped_freeman_abs.urdf (robot description, URDF)
Before this commit: robot balance, 12 links, 11 joints
Links:
- removed link origin
- removed link x_prismatic
- removed link y_prismatic
- removed link z_prismatic
Joints:
- removed joint origin_to_z
- removed joint x_to_y
- removed joint y_to_head
- removed joint z_to_x
