Commit message: 2D TRAINING SETUP AND SAVE FUNCTIONALITY FIXED

File: simulation_env/assets/biped_2d_simple.urdf (robot description, URDF)
Before this commit: robot balance, 8 links, 7 joints
Links:
- added link origin, mass 0; visual box size=0.1 0.1 0.1
- added link x_prismatic, mass 0
- added link y_prismatic, mass 0
- added link z_prismatic, mass 0
Joints:
- added joint origin_to_z: type prismatic, parent origin, child z_prismatic, origin xyz=0 0 0 rpy=0 0 0, axis 0 0 1, limit lower=1 upper=-1 effort=0.0 velocity=1000.0
- added joint x_to_head: type continuous, parent x_prismatic, child head, origin xyz=0 0 0 rpy=0 0 0, axis 1 0 0, limit lower=1 upper=-1 effort=0.0 velocity=1000.0
- added joint y_to_x: type prismatic, parent y_prismatic, child x_prismatic, origin xyz=0 0 0 rpy=0 0 0, axis 1 0 0, limit lower=1 upper=-1 effort=0.0 velocity=1000.0
- added joint z_to_y: type prismatic, parent z_prismatic, child y_prismatic, origin xyz=0 0 0 rpy=0 0 0, axis 0 1 0, limit lower=1 upper=-1 effort=0.0 velocity=1000.0

Commit message: some fixes to model and training

File: simulation_env/assets/biped_2d_simple.urdf (robot description, URDF)
Before this commit: robot balance, 12 links, 11 joints
Joints:
- joint l_ankle: limit lower=-2 upper=2 effort=10.0 velocity=1000.0 -> lower=-0.7 upper=0.7 effort=10.0 velocity=1000.0; type fixed -> revolute
- joint r_ankle: limit lower=-2. upper=2 effort=10.0 velocity=1000.0 -> lower=-0.7 upper=0.7 effort=10.0 velocity=1000.0; type fixed -> revolute
